Commit message: Update robot.urdf

File: src/surveillance_robot_description/urdf/robot.urdf (robot description, URDF)
Before this commit: robot surveillance_robot, 4 links, 3 joints
Links:
- added link camera_optical_frame
- added link caster_wheel, mass 0.5; collision sphere radius=0.05; visual sphere radius=0.05
- link base_link: mass None -> 5.0; geometry collision box size=0.4 0.3 0.1; visual box size=0.4 0.3 0.1
- link left_wheel: mass None -> 0.5; geometry collision cylinder length=0.05 radius=0.1; visual cylinder length=0.05 radius=0.1
- link right_wheel: mass None -> 0.5; geometry collision cylinder length=0.05 radius=0.1; visual cylinder length=0.05 radius=0.1
Joints:
- added joint camera_optical_joint: type fixed, parent camera_link, child camera_optical_frame, origin xyz=0 0 0 rpy=-1.5707 0 -1.5707
- added joint caster_joint: type fixed, parent base_link, child caster_wheel, origin xyz=-0.15 0.0 -0.05
- joint camera_joint: origin xyz=0 0 0.1 -> xyz=0.2 0 0.08 rpy=0 0 0
- joint left_wheel_joint: axis 0 1 0 -> 0 0 1; origin xyz=0 0.15 -0.05 -> xyz=0.0 0.175 0.0 rpy=-1.5707 0 0
- joint right_wheel_joint: axis 0 1 0 -> 0 0 1; origin xyz=0 -0.15 -0.05 -> xyz=0.0 -0.175 0.0 rpy=-1.5707 0 0
